Commit message: feat(mission): basic mission structure

File: src/agv_description/urdf/agv.ros2_control.xacro (robot description, xacro)
@@ -16,30 +16,6 @@
                 <state_interface name="velocity"/>
             </joint>
-            <joint name="base_to_shoulder">
+            <joint name="base_to_fork_lift">
                 <command_interface name="position"/>
-                <state_interface name="position"/>
-                <state_interface name="velocity"/>
-            </joint>
-            <joint name="shoulder_to_upper">
-                <command_interface name="position"/>
-                <state_interface name="position"/>
-                <state_interface name="velocity"/>
-            </joint>
-            <joint name="upper_to_forearm">
-                <command_interface name="position"/>
-                <state_interface name="position"/>
-                <state_interface name="velocity"/>
-            </joint>
-            <joint name="forearm_to_wrist">
-                <command_interface name="position"/>
-                <state_interface name="position"/>
-                <state_interface name="velocity"/>
-            </joint>
-            <joint name="gripper_to_left">
-                <command_interface name="position"/>
-                <state_interface name="position"/>
-                <state_interface name="velocity"/>
-            </joint>
-            <joint name="gripper_to_right">
                 <state_interface name="position"/>
                 <state_interface name="velocity"/>

File: src/agv_description/urdf/agv.urdf.xacro (robot description, xacro)
@@ -6,5 +6,4 @@
     <xacro:include filename="base.urdf.xacro"/>
     <xacro:include filename="wheels.urdf.xacro"/>
-    <xacro:include filename="arm.urdf.xacro"/>
     <xacro:include filename="sensors.urdf.xacro"/>
     <xacro:include filename="agv.ros2_control.xacro"/>
@@ -23,52 +22,68 @@
         <axis xyz="0 1 0"/>
     </joint>
-    <!-- Joints for arm (4-DOF) -->
-    <joint name="base_to_shoulder" type="revolute">
+    <!-- Forklift mast (fixed) -->
+    <link name="mast_link">
+        <visual>
+            <geometry>
+                <box size="0.05 0.25 0.6"/>
+            </geometry>
+            <origin rpy="0 0 0" xyz="0 0 0.3"/>
+            <material name="grey"/>
+        </visual>
+        <collision>
+            <geometry>
+                <box size="0.05 0.25 0.6"/>
+            </geometry>
+            <origin rpy="0 0 0" xyz="0 0 0.3"/>
+        </collision>
+        <inertial>
+            <mass value="3.0"/>
+            <inertia ixx="0.02" ixy="0" ixz="0" iyy="0.02" iyz="0" izz="0.02"/>
+        </inertial>
+    </link>
+    <joint name="base_to_mast" type="fixed">
         <parent link="base_link"/>
-        <child link="shoulder_link"/>
-        <origin xyz="0.2 0 0.1" rpy="0 0 0"/>
+        <child link="mast_link"/>
+        <origin xyz="0.23 0 0.05" rpy="0 0 0"/>
+    </joint>
+    <!-- Fork carriage (prismatic lift) -->
+    <link name="fork_link">
+        <visual>
+            <geometry>
+                <box size="0.35 0.04 0.02"/>
+            </geometry>
+            <origin rpy="0 0 0" xyz="0.17 0.08 0.01"/>
+            <material name="black"/>
+        </visual>
+        <visual>
+            <geometry>
+                <box size="0.35 0.04 0.02"/>
+            </geometry>
+            <origin rpy="0 0 0" xyz="0.17 -0.08 0.01"/>
+            <material name="black"/>
+        </visual>
+        <collision>
+            <geometry>
+                <box size="0.35 0.2 0.02"/>
+            </geometry>
+            <origin rpy="0 0 0" xyz="0.17 0 0.01"/>
+        </collision>
+        <inertial>
+            <mass value="2.0"/>
+            <inertia ixx="0.01" ixy="0" ixz="0" iyy="0.01" iyz="0" izz="0.01"/>
+        </inertial>
+    </link>
+    <joint name="base_to_fork_lift" type="prismatic">
+        <parent link="base_link"/>
+        <child link="fork_link"/>
+        <origin xyz="0.2 0 0.02" rpy="0 0 0"/>
         <axis xyz="0 0 1"/>
-        <limit lower="-1.57" upper="1.57" effort="10" velocity="1"/>
+        <limit lower="0.0" upper="0.15" effort="500.0" velocity="0.15"/>
     </joint>
-    <joint name="shoulder_to_upper" type="revolute">
-        <parent link="shoulder_link"/>
-        <child link="upper_arm_link"/>
-        <origin xyz="0 0 0.1" rpy="0 0 0"/>
-        <axis xyz="0 1 0"/>
-        <limit lower="-1.57" upper="1.57" effort="10" velocity="1"/>
-    </joint>
-    <joint name="upper_to_forearm" type="revolute">
-        <parent link="upper_arm_link"/>
-        <child link="forearm_link"/>
-        <origin xyz="0 0 0.3" rpy="0 0 0"/>
-        <axis xyz="0 1 0"/>
-        <limit lower="-1.57" upper="1.57" effort="10" velocity="1"/>
-    </joint>
-    <joint name="forearm_to_wrist" type="revolute">
-        <parent link="forearm_link"/>
-        <child link="wrist_link"/>
-        <origin xyz="0 0 0.3" rpy="0 0 0"/>
-        <axis xyz="1 0 0"/>
-        <limit lower="-1.57" upper="1.57" effort="5" velocity="1"/>
-    </joint>
-    <joint name="wrist_to_gripper" type="fixed">
-        <parent link="wrist_link"/>
-        <child link="gripper_base"/>
-        <origin xyz="0 0 0.1" rpy="0 0 0"/>
-    </joint>
-    <joint name="gripper_to_left" type="prismatic">
-        <parent link="gripper_base"/>
-        <child link="gripper_left"/>
-        <origin xyz="0 0 0" rpy="0 0 0"/>
-        <axis xyz="1 0 0"/>
-        <limit lower="-0.04" upper="0.04" effort="5" velocity="0.5"/>
-    </joint>
-    <joint name="gripper_to_right" type="prismatic">
-        <parent link="gripper_base"/>
-        <child link="gripper_right"/>
-        <origin xyz="0 0 0" rpy="0 0 0"/>
-        <axis xyz="-1 0 0"/>
-        <limit lower="-0.04" upper="0.04" effort="5" velocity="0.5"/>
-        <mimic joint="gripper_to_left" multiplier="-1" offset="0"/>
+    <link name="fork_tip"/>
+    <joint name="fork_to_tip" type="fixed">
+        <parent link="fork_link"/>
+        <child link="fork_tip"/>
+        <origin xyz="0.35 0 0.02" rpy="0 0 0"/>
     </joint>
     <!-- Joints for caster wheels -->
@@ -94,5 +109,5 @@
         <parent link="base_link"/>
         <child link="camera_link"/>
-        <origin xyz="0.25 0 0.1" rpy="0 0 0"/>
+        <origin xyz="0.22 0 0.35" rpy="0 0 0"/>
     </joint>
 </robot>

File: src/agv_description/urdf/base.urdf.xacro (robot description, xacro)
@@ -19,4 +19,18 @@
             <inertia ixx="0.1" ixy="0" ixz="0" iyy="0.1" iyz="0" izz="0.1"/>
         </inertial>
+        <!-- Camera Pillar -->
+        <visual>
+            <geometry>
+                <cylinder radius="0.02" length="0.3"/>
+            </geometry>
+            <origin rpy="0 0 0" xyz="0.2 0 0.2"/>
+            <material name="grey"/>
+        </visual>
+        <collision>
+            <geometry>
+                <cylinder radius="0.02" length="0.3"/>
+            </geometry>
+            <origin rpy="0 0 0" xyz="0.2 0 0.2"/>
+        </collision>
     </link>
 </robot>
