Commit message: Integrate controllers and gazebo launch

File: src/agv_description/urdf/agv.urdf.xacro (robot description, xacro)
@@ -2,4 +2,5 @@
 <robot name="agv"
     xmlns:xacro="http://www.ros.org/wiki/xacro">
+    <xacro:arg name="controller_config" default=""/>
     <xacro:include filename="materials.urdf.xacro"/>
     <xacro:include filename="base.urdf.xacro"/>
@@ -7,4 +8,6 @@
     <xacro:include filename="arm.urdf.xacro"/>
     <xacro:include filename="sensors.urdf.xacro"/>
+    <xacro:include filename="agv.ros2_control.xacro"/>
+    <xacro:agv_ros2_control controller_config="$(arg controller_config)"/>
     <!-- Joints for wheels -->
     <joint name="base_to_left_wheel" type="continuous">
@@ -67,15 +70,18 @@
         <axis xyz="-1 0 0"/>
         <limit lower="-0.04" upper="0.04" effort="5" velocity="0.5"/>
+        <mimic joint="gripper_to_left" multiplier="-1" offset="0"/>
     </joint>
     <!-- Joints for caster wheels -->
-    <joint name="base_to_caster_front" type="fixed">
+    <joint name="base_to_caster_front" type="continuous">
         <parent link="base_link"/>
         <child link="caster_front"/>
-        <origin xyz="0.2 0 -0.04" rpy="0 0 0"/>
+        <origin xyz="0.2 0 0.03" rpy="0 0 0"/>
+        <axis xyz="0 1 0"/>
     </joint>
-    <joint name="base_to_caster_rear" type="fixed">
+    <joint name="base_to_caster_rear" type="continuous">
         <parent link="base_link"/>
         <child link="caster_rear"/>
-        <origin xyz="-0.2 0 -0.04" rpy="0 0 0"/>
+        <origin xyz="-0.2 0 0.03" rpy="0 0 0"/>
+        <axis xyz="0 1 0"/>
     </joint>
     <!-- Joints for sensors -->

File: src/agv_description/urdf/wheels.urdf.xacro (robot description, xacro)
@@ -39,20 +39,22 @@
         </inertial>
     </link>
-    <!-- Caster wheels -->
+    <!-- Caster wheels (small rolling wheels) -->
     <link name="caster_front">
         <visual>
             <geometry>
-                <sphere radius="0.04"/>
+                <cylinder radius="0.03" length="0.02"/>
             </geometry>
+            <origin rpy="1.5708 0 0" xyz="0 0 0"/>
             <material name="grey"/>
         </visual>
         <collision>
             <geometry>
-                <sphere radius="0.04"/>
+                <cylinder radius="0.03" length="0.02"/>
             </geometry>
+            <origin rpy="1.5708 0 0" xyz="0 0 0"/>
         </collision>
         <inertial>
             <mass value="0.2"/>
-            <inertia ixx="0.002" ixy="0" ixz="0" iyy="0.002" iyz="0" izz="0.002"/>
+            <inertia ixx="0.001" ixy="0" ixz="0" iyy="0.001" iyz="0" izz="0.001"/>
         </inertial>
     </link>
@@ -60,16 +62,18 @@
         <visual>
             <geometry>
-                <sphere radius="0.04"/>
+                <cylinder radius="0.03" length="0.02"/>
             </geometry>
+            <origin rpy="1.5708 0 0" xyz="0 0 0"/>
             <material name="grey"/>
         </visual>
         <collision>
             <geometry>
-                <sphere radius="0.04"/>
+                <cylinder radius="0.03" length="0.02"/>
             </geometry>
+            <origin rpy="1.5708 0 0" xyz="0 0 0"/>
         </collision>
         <inertial>
             <mass value="0.2"/>
-            <inertia ixx="0.002" ixy="0" ixz="0" iyy="0.002" iyz="0" izz="0.002"/>
+            <inertia ixx="0.001" ixy="0" ixz="0" iyy="0.001" iyz="0" izz="0.001"/>
         </inertial>
     </link>

Commit message: feat(navigation): Nav2 and SLAM integration

File: src/agv_description/urdf/agv.urdf.xacro (robot description, xacro)
@@ -14,5 +14,5 @@
         <parent link="base_link"/>
         <child link="left_wheel"/>
-        <origin xyz="-0.15 0.2 0.05" rpy="0 0 0"/>
+        <origin xyz="-0.15 0.2 0.1" rpy="0 0 0"/>
         <axis xyz="0 1 0"/>
     </joint>
@@ -20,5 +20,5 @@
         <parent link="base_link"/>
         <child link="right_wheel"/>
-        <origin xyz="-0.15 -0.2 0.05" rpy="0 0 0"/>
+        <origin xyz="-0.15 -0.2 0.1" rpy="0 0 0"/>
         <axis xyz="0 1 0"/>
     </joint>

File: src/agv_description/urdf/wheels.urdf.xacro (robot description, xacro)
@@ -14,4 +14,5 @@
                 <cylinder radius="0.1" length="0.05"/>
             </geometry>
+            <origin rpy="1.5708 0 0" xyz="0 0 0"/>
         </collision>
         <inertial>
@@ -33,4 +34,5 @@
                 <cylinder radius="0.1" length="0.05"/>
             </geometry>
+            <origin rpy="1.5708 0 0" xyz="0 0 0"/>
         </collision>
         <inertial>

Commit message: feat(mission): implement complete autonomous mission system and fix nav2 configs

File: src/agv_description/urdf/agv.urdf.xacro (robot description, xacro)
@@ -14,5 +14,5 @@
         <parent link="base_link"/>
         <child link="left_wheel"/>
-        <origin xyz="-0.15 0.2 0.1" rpy="0 0 0"/>
+        <origin xyz="-0.15 0.2 0.0" rpy="0 0 0"/>
         <axis xyz="0 1 0"/>
     </joint>
@@ -20,5 +20,5 @@
         <parent link="base_link"/>
         <child link="right_wheel"/>
-        <origin xyz="-0.15 -0.2 0.1" rpy="0 0 0"/>
+        <origin xyz="-0.15 -0.2 0.0" rpy="0 0 0"/>
         <axis xyz="0 1 0"/>
     </joint>
@@ -76,5 +76,5 @@
         <parent link="base_link"/>
         <child link="caster_front"/>
-        <origin xyz="0.2 0 0.03" rpy="0 0 0"/>
+        <origin xyz="0.2 0 -0.07" rpy="0 0 0"/>
         <axis xyz="0 1 0"/>
     </joint>
@@ -82,5 +82,5 @@
         <parent link="base_link"/>
         <child link="caster_rear"/>
-        <origin xyz="-0.2 0 0.03" rpy="0 0 0"/>
+        <origin xyz="-0.2 0 -0.07" rpy="0 0 0"/>
         <axis xyz="0 1 0"/>
     </joint>

File: src/agv_description/urdf/base.urdf.xacro (robot description, xacro)
@@ -13,4 +13,5 @@
                 <box size="0.5 0.3 0.1"/>
             </geometry>
+            <origin rpy="0 0 0" xyz="0 0 0.05"/>
         </collision>
         <inertial>

File: src/agv_description/urdf/wheels.urdf.xacro (robot description, xacro)
@@ -80,3 +80,13 @@
         </inertial>
     </link>
+    <gazebo reference="caster_front">
+        <mu1>0.0</mu1>
+        <mu2>0.0</mu2>
+        <material>Gazebo/Grey</material>
+    </gazebo>
+    <gazebo reference="caster_rear">
+        <mu1>0.0</mu1>
+        <mu2>0.0</mu2>
+        <material>Gazebo/Grey</material>
+    </gazebo>
 </robot>

Commit message: feat(mission): update mission controller to use TwistStamped and resolve flake8 style issues

File: src/agv_description/urdf/agv.urdf.xacro (robot description, xacro)
@@ -79,5 +79,5 @@
         <origin xyz="0.2 0 0.02" rpy="0 0 0"/>
         <axis xyz="0 0 1"/>
-        <limit lower="0.0" upper="0.15" effort="500.0" velocity="0.15"/>
+        <limit lower="0.0" upper="0.35" effort="500.0" velocity="0.15"/>
     </joint>
     <link name="fork_tip"/>
@@ -109,5 +109,5 @@
         <parent link="base_link"/>
         <child link="camera_link"/>
-        <origin xyz="0.22 0 0.35" rpy="0 0 0"/>
+        <origin xyz="0.28 0 0.40" rpy="0 0 0"/>
     </joint>
 </robot>

File: src/agv_description/urdf/sensors.urdf.xacro (robot description, xacro)
@@ -10,14 +10,15 @@
             <material name="black"/>
         </visual>
+        <inertial>
+            <mass value="0.1"/>
+            <inertia ixx="1e-4" ixy="0" ixz="0" iyy="1e-4" iyz="0" izz="1e-4"/>
+        </inertial>
     </link>
     <!-- Camera -->
     <link name="camera_link">
-        <visual>
-            <geometry>
-                <box size="0.03 0.05 0.02"/>
-            </geometry>
-            <origin rpy="0 0 0" xyz="0 0 0"/>
-            <material name="black"/>
-        </visual>
+        <inertial>
+            <mass value="0.05"/>
+            <inertia ixx="1e-5" ixy="0" ixz="0" iyy="1e-5" iyz="0" izz="1e-5"/>
+        </inertial>
     </link>
     <gazebo reference="lidar_link">
@@ -33,5 +34,5 @@
                 </scan>
                 <range>
-                    <min>0.05</min>
+                    <min>0.45</min>
                     <max>10.0</max>
                 </range>
@@ -46,5 +47,5 @@
             <update_rate>30</update_rate>
             <camera>
-                <horizontal_fov>1.0472</horizontal_fov>
+                <horizontal_fov>1.5708</horizontal_fov>
                 <image>
                     <width>640</width>

Commit message: done

File: src/agv_description/urdf/agv.urdf.xacro (robot description, xacro)
@@ -63,10 +63,4 @@
             <material name="black"/>
         </visual>
-        <collision>
-            <geometry>
-                <box size="0.35 0.2 0.02"/>
-            </geometry>
-            <origin rpy="0 0 0" xyz="0.17 0 0.01"/>
-        </collision>
         <inertial>
             <mass value="2.0"/>
@@ -111,3 +105,27 @@
         <origin xyz="0.28 0 0.40" rpy="0 0 0"/>
     </joint>
+    <!-- Gazebo DetachableJoint plugins for picking up cargo -->
+    <gazebo>
+        <plugin filename="gz-sim-detachable-joint-system" name="gz::sim::systems::DetachableJoint">
+            <parent_link>fork_link</parent_link>
+            <child_model>cargo_red_1</child_model>
+            <child_model_link>link</child_model_link>
+            <detach_topic>/model/agv/detach_red</detach_topic>
+            <attach_topic>/model/agv/attach_red</attach_topic>
+        </plugin>
+        <plugin filename="gz-sim-detachable-joint-system" name="gz::sim::systems::DetachableJoint">
+            <parent_link>fork_link</parent_link>
+            <child_model>cargo_blue_1</child_model>
+            <child_model_link>link</child_model_link>
+            <detach_topic>/model/agv/detach_blue</detach_topic>
+            <attach_topic>/model/agv/attach_blue</attach_topic>
+        </plugin>
+        <plugin filename="gz-sim-detachable-joint-system" name="gz::sim::systems::DetachableJoint">
+            <parent_link>fork_link</parent_link>
+            <child_model>cargo_yellow_1</child_model>
+            <child_model_link>link</child_model_link>
+            <detach_topic>/model/agv/detach_yellow</detach_topic>
+            <attach_topic>/model/agv/attach_yellow</attach_topic>
+        </plugin>
+    </gazebo>
 </robot>

File: src/agv_description/urdf/sensors.urdf.xacro (robot description, xacro)
@@ -34,5 +34,5 @@
                 </scan>
                 <range>
-                    <min>0.45</min>
+                    <min>0.48</min>
                     <max>10.0</max>
                 </range>

File: src/agv_description/urdf/wheels.urdf.xacro (robot description, xacro)
@@ -80,4 +80,18 @@
         </inertial>
     </link>
+    <gazebo reference="left_wheel">
+        <mu1>1.0</mu1>
+        <mu2>1.0</mu2>
+        <kp>10000000.0</kp>
+        <kd>1.0</kd>
+        <material>Gazebo/Black</material>
+    </gazebo>
+    <gazebo reference="right_wheel">
+        <mu1>1.0</mu1>
+        <mu2>1.0</mu2>
+        <kp>10000000.0</kp>
+        <kd>1.0</kd>
+        <material>Gazebo/Black</material>
+    </gazebo>
     <gazebo reference="caster_front">
         <mu1>0.0</mu1>
